File: hardware/eagle/HAN_DE10-Lite_PS2SpeakerShield_001.sch (EAGLE design)
At the start: 20 parts

Commit message: Update hardware documentation
Other:
- moved on the sheet: B1, C1, C2, C3, C4, D1, D2, D3, D4, LS1, R1, R2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
