File: hardware/kicad/HAN_DE10-Lite_PS2SpeakerShield_010/HAN_DE10-Lite_PS2SpeakerShield_001.kicad_pcb (KiCad board)
At the start: 2 copper layers, 53.3 x 59.7 mm, 21 parts

Commit message: Updated documentation
Routing:
- net MSCLK: track 17.3 -> 19.1 mm
Changed lines of the file:
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@@
     (descr "<li><b>SOT23</b><hr> <ul><li>Plastic surface-mounted package; 3 leads<li><u>JEDEC</u>: TO-236AB <li><u>IEC</u>: -- <li><u>JEITA</u>: --</ul>")
     (fp_text reference "D4" (at 0.7239 4.2164 90) (layer "F.SilkS")
-        (effects (font (size 0.9264 0.9264) (thickness 0.0736)) (justify left bottom))
+        (effects (font (size 0.9264 0.9264) (thickness 0.1)) (justify left bottom))
     )
     (fp_text value "BAT54S" (at 2.5 1) (layer "F.Fab") hide
@@
     (descr "<li><b>SOT23</b><hr> <ul><li>Plastic surface-mounted package; 3 leads<li><u>JEDEC</u>: TO-236AB <li><u>IEC</u>: -- <li><u>JEITA</u>: --</ul>")
     (fp_text reference "D2" (at 0.7239 4.2164 90) (layer "F.SilkS")
-        (effects (font (size 0.9264 0.9264) (thickness 0.0736)) (justify left bottom))
+        (effects (font (size 0.9264 0.9264) (thickness 0.1)) (justify left bottom))
     )
     (fp_text value "BAT54S" (at 2.5 1) (layer "F.Fab") hide
@@
     (descr "<b>CAPACITOR</b>")
     (fp_text reference "C3" (at 2.794 0.508 90) (layer "F.SilkS")
-        (effects (font (size 1.176528 1.176528) (thickness 0.093472)) (justify right top))
+        (effects (font (size 1.176528 1.176528) (thickness 0.1)) (justify right top))
     )
     (fp_text value "100n" (at -1.27 2.54 -90) (layer "F.Fab") hide
@@
     (descr "<li><b>SOT23</b><hr> <ul><li>Plastic surface-mounted package; 3 leads<li><u>JEDEC</u>: TO-236AB <li><u>IEC</u>: -- <li><u>JEITA</u>: --</ul>")
     (fp_text reference "D1" (at 0.7239 4.2164 90) (layer "F.SilkS")
-        (effects (font (size 0.9264 0.9264) (thickness 0.0736)) (justify left bottom))
+        (effects (font (size 0.9264 0.9264) (thickness 0.1)) (justify left bottom))
     )
     (fp_text value "BAT54S" (at 2.5 1) (layer "F.Fab") hide
@@
     (descr "<li><b>SOT23</b><hr> <ul><li>Plastic surface-mounted package; 3 leads<li><u>JEDEC</u>: TO-236AB <li><u>IEC</u>: -- <li><u>JEITA</u>: --</ul>")
     (fp_text reference "D3" (at 0.7239 4.2164 90) (layer "F.SilkS")
-        (effects (font (size 0.9264 0.9264) (thickness 0.0736)) (justify left bottom))
+        (effects (font (size 0.9264 0.9264) (thickness 0.1)) (justify left bottom))
     )
     (fp_text value "BAT54S" (at 2.5 1) (layer "F.Fab") hide
@@
   (segment (start 142.1511 91.6686) (end 142.1511 95.4786) (width 0.254) (layer "B.Cu") (net 7))
   (segment (start 142.1511 95.4786) (end 140.8811 96.7486) (width 0.254) (layer "B.Cu") (net 7))
+  (segment (start 140.8811 90.3986) (end 142.1511 91.6686) (width 0.254) (layer "B.Cu") (net 7))
   (segment (start 142.2111 83.9886) (end 143.4211 82.7786) (width 0.254) (layer "F.Cu") (net 8))
   (segment (start 148.5011 91.5386) (end 148.6311 91.6686) (width 0.254) (layer "F.Cu") (net 8))

Commit message: Remove PII from various project files
Removed names, email addresses, student numbers, and initials from README.md, .vhd, and .kicad_pcb files throughout the repository to protect personal information.
Other:
- board text added: "20240320 [Redacted]"
- board text removed: "20240320 WLGRW"
Changed lines of the file:
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@@
   (gr_line (start 121.8311 132.3086) (end 124.3711 132.3086)
     (stroke (width 0.05) (type solid)) (layer "Edge.Cuts"))
-  (gr_text "20240320 WLGRW" (at 127.635 132.715) (layer "F.SilkS")
+  (gr_text "20240320 [Redacted]" (at 127.635 132.715) (layer "F.SilkS")
     (effects (font (size 1.194816 1.194816) (thickness 0.227584)) (justify left bottom))
   )
